Commit message: sla

File: followyollo_simulation/urdf/followyolo.urdf.xacro (robot description, xacro)
@@ -189,5 +189,5 @@
     <parent link="base_link"/>
     <child link="basket_link"/>
-    <origin xyz="-0.08 0.0 0.24" rpy="0 0 0"/>
+    <origin xyz="-0.08 0.0 0.3" rpy="0 0 0"/>
     <axis xyz="0 0 1"/>
   </joint>
