Commit message: modificações nos .launch e .xacro e mudança para Pose

File: followyollo_simulation/urdf/person.urdf.xacro (robot description, xacro)
@@ -4,4 +4,5 @@
   <xacro:include filename="$(find turtlebot3_description)/urdf/turtlebot3_waffle_pi.gazebo.xacro"/>
   <xacro:arg name="artag" default="package://followyollo_simulation/meshes/ARTag0.dae"/>
+  <xacro:arg name="isUser" default="false"/>
   <link name="base_footprint"/>
   <joint name="base_joint" type="fixed">
@@ -16,5 +17,4 @@
         <mesh filename="package://followyollo_simulation/meshes/pessoa.stl" scale="0.1 0.1 0.1"/>
       </geometry>
-      <material name="light_black"/>
     </visual>
     <collision>
@@ -32,4 +32,9 @@
     </inertial>
   </link>
+  <xacro:if value="$(arg isUser)">
+    <gazebo reference="base_link">
+      <material>Gazebo/Blue</material>
+    </gazebo>
+  </xacro:if>
   <joint name="artag1_joint" type="fixed">
     <parent link="base_link"/>
